File: eagle/K104.brd (EAGLE design)
At the start: 428.3 x 123.6 mm, 229 parts, among them IC1 MAX7219CNG, IC2 MAX7219CNG

Commit message: add PCB and case files
Parts:
- added U$2, U$3: (no value), oshw:OSHW_8MM
